Commit message: implemented flc

File: urdf/planar2dof.urdf (robot description, URDF)
Before this commit: robot planar2dof, 5 links, 4 joints
Links:
- link planar2dof/link_striker_ee: mass 0.1 -> 1.3

Commit message: polynomial trajectory

File: urdf/planar2dof.urdf (robot description, URDF)
Before this commit: robot planar2dof, 5 links, 4 joints
Links:
- link planar2dof/link_striker_ee: mass 1.3 -> 1.2

Commit message: before mma

File: urdf/planar2dof.urdf (robot description, URDF)
Before this commit: robot planar2dof, 5 links, 4 joints
Links:
- link planar2dof/link_striker_ee: mass 1.2 -> 0.1
